File: hardware/hardware.kicad_pcb (KiCad board)
At the start: 2 copper layers, 21 parts, among them J1 USB_B_Micro, J3 Conn_02x05_Odd_Even, J4 Conn_02x03_Odd_Even, U1 HY931147C, U28 CH32V307RCT6, U3 LM1117-3.3, U4 CH340C, Y1 Crystal_GND24

Commit message: differencial wiring
Parts:
- removed J4: Conn_02x03_Odd_Even, Connector_PinHeader_2.54mm:PinHeader_2x03_P2.54mm_Vertical
- removed R31, R32: R_Small, Resistor_SMD:R_0603_1608Metric
- added JP1: Jumper_3_Open, Jumper:SolderJumper-3_P1.3mm_Open_RoundedPad1.0x1.5mm, F.Cu at (156.7, 41.0)
- added JP2: Jumper_3_Open, Jumper:SolderJumper-3_P1.3mm_Open_RoundedPad1.0x1.5mm, F.Cu at (161.7, 41.0)
- J3: footprint Connector_PinHeader_2.54mm:PinHeader_2x05_P2.54mm_Vertical -> Connector_JST:JST_SH_BM10B-SRSS-TB_1x10-1MP_P1.00mm_Vertical
- moved R1 42.6 mm to (136.0, 41.4)
- moved Y1 38.1 mm to (158.3, 49.1), turned to -90 degrees
- moved D25 32.8 mm to (140.0, 43.0), turned to 180 degrees
- moved R2 32.6 mm to (132.0, 59.8)
- moved J3 30.3 mm to (153.7, 60.3), turned to 180 degrees
- moved R54 27.4 mm to (140.0, 41.5)
- moved J1 27.0 mm to (167.2, 46.0), turned to 90 degrees
- moved C4 25.7 mm to (165.5, 51.5), turned to 180 degrees
- moved U4 24.3 mm to (165.5, 58.0)
- moved C7 22.8 mm to (154.5, 53.5)
- moved C1 19.3 mm to (158.0, 45.0)
- moved C2 15.9 mm to (158.0, 53.0), turned to 180 degrees
- moved U3 12.9 mm to (141.3, 59.5)
- moved C6 10.8 mm to (141.7, 52.5), turned to 180 degrees
- moved C5 10.6 mm to (138.5, 54.5)
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- renumbered U28 to U1
Connections:
- U1 pad 29: SCL -> unconnected-(U28-PB10-Pad29)
- U1 pad 30: SDA -> unconnected-(U28-PB11-Pad30)
Routing:
- net D+: track 0.00 -> 17.3 mm
- net D-: track 0.00 -> 17.3 mm
- net TD_N: track 0.00 -> 12.7 mm
- net TD_P: track 0.00 -> 12.6 mm
- net RD_N: track 0.00 -> 11.0 mm
- net RD_P: track 0.00 -> 10.9 mm
- net XTAL2: track 0.00 -> 8.53 mm
- net XTAL1: track 0.00 -> 5.93 mm
- net +3V3: track 0.00 -> 4.27 mm

Commit message: wiring pcb
Parts:
- added J2: Conn_01x08, Connector_JST:JST_SH_BM08B-SRSS-TB_1x08-1MP_P1.00mm_Vertical, F.Cu at (153.4, 60.4)
- J3: value Conn_02x05_Odd_Even -> Conn_01x04; footprint Connector_JST:JST_SH_BM10B-SRSS-TB_1x10-1MP_P1.00mm_Vertical -> Connector_PinHeader_2.54mm:PinHeader_1x04_P2.54mm_Vertical
- moved J3 32.0 mm to (121.8, 62.4), turned to 90 degrees
- moved C5 10.8 mm to (149.0, 57.0)
- moved C3 0.50 mm to (136.0, 61.0)
- renumbered U1 to U28
Connections:
- J3 pad 1: SWCLK -> V-
- J3 pad 2: TX-PROG -> V+
- J3 pad 3: SWDIO -> GND
- J3 pad 4: RX-PROG -> +3V3
Routing:
- net +5V: track 0.00 -> 44.5 mm, vias 0 -> 2
- net GND: track 0.00 -> 38.2 mm, vias 0 -> 22
- net LED2: track 0.00 -> 36.5 mm, vias 0 -> 1
- net +3V3: track 4.27 -> 35.0 mm, vias 0 -> 53
- net V+: track 0.00 -> 30.7 mm
- net RX-PROG: track 0.00 -> 30.4 mm, vias 0 -> 2
- net LED1: track 0.00 -> 29.8 mm
- net TX-PROG: track 0.00 -> 28.0 mm, vias 0 -> 2
- net V-: track 0.00 -> 26.1 mm
- net BOOT0: track 0.00 -> 19.3 mm, vias 0 -> 2
- net BOOT1: track 0.00 -> 17.8 mm, vias 0 -> 2
- net SWDIO: track 0.00 -> 15.2 mm
- net Net-(U1-Y+): track 0.00 -> 14.7 mm
- net Net-(U1-G+): track 0.00 -> 13.3 mm
- net RST: track 0.00 -> 12.7 mm, vias 0 -> 2
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- added copper zone on B.Cu, net +3V3
- added copper zone on F.Cu, net +3V3
- added copper zone on In2.Cu, net +3V3
- added copper zone on F.Cu, net GND
- added copper zone on In1.Cu, net GND
Other:
- board outline added: 52.5 x 26 mm
- copper layers 2 -> 4
