File: hardware/hardware.kicad_sch (KiCad schematic)
At the start: 21 parts, among them J1 USB_B_Micro, J3 Conn_02x05_Odd_Even, J4 Conn_02x03_Odd_Even, U1 HY931147C, U28 CH32V307RCT6, U3 LM1117-3.3, U4 CH340C, Y1 Crystal_GND24

Commit message: differencial wiring
Parts:
- removed J4: Conn_02x03_Odd_Even, Connector_PinHeader_2.54mm:PinHeader_2x03_P2.54mm_Vertical, symbol Connector_Generic:Conn_02x03_Odd_Even
- removed R31, R32: R_Small, Resistor_SMD:R_0603_1608Metric, symbol Device:R_Small
- added JP1, JP2: Jumper_3_Open, Jumper:SolderJumper-3_P1.3mm_Open_RoundedPad1.0x1.5mm, symbol Jumper:Jumper_3_Open
- J3: footprint Connector_PinHeader_2.54mm:PinHeader_2x05_P2.54mm_Vertical -> Connector_JST:JST_SH_BM10B-SRSS-TB_1x10-1MP_P1.00mm_Vertical
Connections:
- net +3V3: now also JP1.1 (A), JP2.1 (A)
- net BOOT0: now also JP2.2 (C)
- net BOOT1: now also JP1.2 (C)
- net GND: now also JP1.3 (B), JP2.3 (B)
- net SCL: no longer names the net of U28.29 (PB10)
- net SDA: no longer names the net of U28.30 (PB11)

Commit message: wiring pcb
Parts:
- removed J3: Conn_02x05_Odd_Even, Connector_JST:JST_SH_BM10B-SRSS-TB_1x10-1MP_P1.00mm_Vertical, symbol Connector_Generic:Conn_02x05_Odd_Even
- added J2: Conn_01x08, Connector_JST:JST_SH_BM08B-SRSS-TB_1x08-1MP_P1.00mm_Vertical, symbol Connector_Generic:Conn_01x08
- added J3: Conn_01x04, Connector_PinHeader_2.54mm:PinHeader_1x04_P2.54mm_Vertical, symbol Connector_Generic:Conn_01x04
Connections:
- net +3V3: now also J2.1 (Pin_1), J3.4 (Pin_4)
- net GND: now also J2.2 (Pin_2), J3.3 (Pin_3)
- net RST: now also J2.4 (Pin_4)
- net RX-PROG: now also J2.5 (Pin_5)
- net SWCLK: now also J2.7 (Pin_7)
- net SWDIO: now also J2.8 (Pin_8)
- net TX-PROG: now also J2.6 (Pin_6)
- net V+: now also J3.2 (Pin_2)
- net V-: now also J3.1 (Pin_1)
